File: connector_usb.kicad_sch (KiCad schematic)
At the start: 11 parts, among them J11 USB C 2.0, U1 USBLC6-2SC6

Commit message: Final edits before sending to fab
Parts:
- renumbered R2 to R4, R3 to R5, R4 to R6, R5 to R7, R6 to R8
