File: debug_leds.kicad_sch (KiCad schematic)
At the start: 16 parts, among them Q2 2N7002, Q3 2N7002, Q4 2N7002, Q5 2N7002, SW4 USR

Commit message: Final edits before sending to fab
Parts:
- renumbered R24 to R27, R25 to R28, R26 to R29, R27 to R30, R28 to R31
