File: imu_lsm6dsv.kicad_sch (KiCad schematic)
At the start: 4 parts, among them U9 M24C64-RMN6TP

Commit message: Final edits before sending to fab
Parts:
- removed C45: 100nF, Capacitor_SMD:C_0603_1608Metric, symbol Device:C_Small_US
- removed R32, R33: 3.3k, Resistor_SMD:R_0603_1608Metric, symbol Device:R_Small_US
- removed U9: M24C64-RMN6TP, Package_SO:SOIC-8_3.9x4.9mm_P1.27mm, symbol Memory_EEPROM:M24C02-RMN
- added C31, C32: 100nF, Capacitor_SMD:C_0603_1608Metric, symbol Device:C_Small_US
- added R16: 10k, Resistor_SMD:R_0603_1608Metric, symbol Device:R_Small_US
- added U6: LSM6DSV, Package_LGA:LGA-14_3x2.5mm_P0.5mm_LayoutBorder3x4y, symbol integrated_motor_controller_lib:LSM6DSV
Connections:
- net +3.3V: now also C31.1, C32.1, R16.1, U6.5 (VDDIO), U6.8 (VDD)
- net GND: now also C31.2, C32.2, U6.2 (SDX), U6.3 (SCX), U6.6 (GND), U6.7 (GND)
- new net IMU_INT1: U6.4 (INT1)
- new net IMU_INT2: U6.9 (INT2)
- new net SPI_CS: R16.2, U6.12 (CS)
- new net SPI_MISO: U6.1 (SDO/SA0)
- new net SPI_MOSI: U6.14 (SDA)
- new net SPI_SCK: U6.13 (SCL)
- no-connect marks 0 -> 2
Other:
- note removed: "BYPASS Capacitor"
- note removed: "E0, E1, E2 Control the lower 3 bits of the I2C address Floating is read as GND Address is 0b1010000(RW bit as LSB) Read: 0xA0 Write: 0xA1"
- company: Designed by: Kyle Gieselman -> (none)
- title: Integrated Motor Controller -> (none)
