File: integrated_motor_controller.kicad_pcb (KiCad board)
At the start: 4 copper layers, 85 x 54 mm, 148 parts, among them J1 RCVR, J10 CH2, J11 USB C 2.0, J12 VMeter, J13 BATT_IN, J14 MOT, J15 MOT, J2 SWD, J3 ENC 0, J4 ENC 1, J5 UART, J6 CH0, J7 I2C, J8 CH1, J9 I2C, Q1 SI7157DP, Q2 2N7002, Q3 2N7002, Q4 2N7002, Q5 2N7002, SW1 SW_PWR, SW2 ~{RST}, SW3 BOOT, SW4 USR, U1 USBLC6-2SC6, U2 AP63205WU, U3 AP1117-33, U4 AP63205WU, U5 STM32H563RITx, U6 ICM-42688-P, U7 DRV8874PWPR, U8 DRV8874PWPR, U9 M24C64-RMN6TP, Y1 ASE-25.000MHZ

Commit message: Final edits before sending to fab
Parts:
- removed the C33 at (132.4, 51.2)
- added R16: 10k, Resistor_SMD:R_0603_1608Metric, F.Cu at (135.4, 53.5)
- added R2: 3.3k, Resistor_SMD:R_0603_1608Metric, F.Cu at (153.2, 76.1)
- added R3: 3.3k, Resistor_SMD:R_0603_1608Metric, F.Cu at (154.7, 78.1)
- C31: value 2.2uF -> 100nF
- U6: value ICM-42688-P -> LSM6DSV; footprint icm-42688:icm-42688 -> Package_LGA:LGA-14_3x2.5mm_P0.5mm_LayoutBorder3x4y
- moved C31 3.66 mm to (132.5, 51.3), turned to 180 degrees
- moved C32 1.67 mm to (130.0, 53.2)
- renumbered C34 to C33, C35 to C34, C36 to C35, C37 to C36, C38 to C37, C39 to C38, C40 to C39, C41 to C40, C42 to C41, C43 to C42, C44 to C43, C45 to C44, C46 to C45, R8 to R10, R9 to R11, R10 to R12, R11 to R13, R12 to R14, R13 to R15, R14 to R17, R15 to R18, R16 to R19, R17 to R20, R18 to R21, R19 to R22, R20 to R23, R21 to R24, R22 to R25, R23 to R26, R24 to R27, R25 to R28, R26 to R29, R27 to R30, R28 to R31, R29 to R32, R30 to R33, R2 to R4, R3 to R5, R4 to R6, R5 to R7, R6 to R8, R7 to R9
Connections:
- U6 pad 11: GND -> unconnected-(U6-SDO_Aux-Pad11)
- U6 pad 2: unconnected-(U6-RESV_2-Pad2) -> GND
- U6 pad 3: unconnected-(U6-RESV_3-Pad3) -> GND
Routing:
- net /IMU/SPI_CS: track 11.7 -> 13.1 mm
- net +3.3V: track 71.8 -> 73.1 mm, vias 26 -> 29
- net /IMU/IMU_INT2: track 12.3 -> 12.0 mm, vias 2 -> 0
- net GND: track 119.4 -> 119.7 mm, vias 78 -> 76
- net Net-(U5-BOOT0): vias 0 -> 2
