File: mcu_h563r.kicad_sch (KiCad schematic)
At the start: 25 parts, among them SW2 ~{RST}, SW3 BOOT, U5 STM32H563RITx, Y1 ASE-25.000MHZ

Commit message: Final edits before sending to fab
Parts:
- renumbered R11 to R13, R12 to R14, R13 to R15
