File: motor_driver_drv8874.kicad_sch (KiCad schematic)
At the start: 13 parts, among them J14 MOT, U7 DRV8874PWPR

Commit message: Final edits before sending to fab
Parts:
- renumbered C34 to C33, C35 to C34, C36 to C35, C37 to C36, C38 to C37, C39 to C38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
