File: power_regulator_2s_3s.kicad_sch (KiCad schematic)
At the start: 36 parts, among them J12 VMeter, J13 BATT_IN, Q1 SI7157DP, SW1 SW_PWR, U2 AP63205WU, U3 AP1117-33, U4 AP63205WU

Commit message: Final edits before sending to fab
Parts:
- renumbered R8 to R10, R9 to R11, R10 to R12, R7 to R9
